File: hardware/buck.brd (EAGLE design)
At the start: 38 x 23 mm, 11 parts, among them X1 MOLEX_4HORIZONTAL

Commit message: move silkscreen labels
Parts:
- IC1: value (none) -> LM2675M-ADJ
- L2: value DR125 -> 68uH 1.5A
Changed lines of the file:
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@@
 <layer number="49" name="Reference" color="7" fill="1" visible="no" active="yes"/>
 <layer number="50" name="dxf" color="7" fill="1" visible="no" active="no"/>
-<layer number="51" name="tDocu" color="7" fill="1" visible="no" active="yes"/>
+<layer number="51" name="tDocu" color="7" fill="1" visible="yes" active="yes"/>
 <layer number="52" name="bDocu" color="7" fill="1" visible="no" active="yes"/>
 <layer number="53" name="tGND_GNDA" color="7" fill="9" visible="no" active="no"/>
@@
 </autorouter>
 <elements>
-<element name="IC1" library="Simplex-ICs" package="SO-08" value="" x="19.1" y="11.5"/>
+<element name="IC1" library="Simplex-ICs" package="SO-08" value="LM2675M-ADJ" x="19.1" y="11.5"/>
 <element name="R1" library="rcl" package="R0805W" value="1.5K 1%" x="21.2" y="5.9" rot="R180"/>
 <element name="R2" library="rcl" package="R0805W" value="4.75k 1%" x="17" y="5.9" rot="R180"/>
@@
 <element name="C2" library="rcl" package="PANASONIC_F" value="47uF, 63V" x="26.6" y="15.6" rot="R90"/>
 <element name="C3" library="rcl" package="PANASONIC_D" value="100uF, 16V" x="26.7" y="5.8" rot="R270"/>
-<element name="L2" library="inductors" package="DR125" value="DR125" x="7.2" y="10.2" rot="R270"/>
+<element name="L2" library="inductors" package="DR125" value="68uH 1.5A" x="7.2" y="10.2" rot="R270"/>
 <element name="JP1" library="SparkFun-Connectors" package="1X02" value="M02PTH" x="35.8" y="14" rot="R180"/>
 <element name="X1" library="Simplex-Connectors" package="0530480401" value="MOLEX_4HORIZONTAL" x="32.2" y="8"/>

Commit message: latest
Parts:
- removed R3: 100k DNP, rcl:R0805W
- removed X1: MOLEX_4HORIZONTAL, Simplex-Connectors:0530480401
- added X2: MKDSN1,5/4-5,08, con-phoenix-508:MKDSN1,5/4-5,08
- JP1: value M02PTH -> M01PTH; device SparkFun-Connectors:1X02 -> SparkFun-Connectors:1X01
- moved JP1 14.2 mm to (29.1, 1.50), turned to 0 degrees
- moved C3 0.60 mm to (26.1, 5.80)
- moved R1 0.50 mm to (20.7, 5.90)
- moved R2 0.50 mm to (16.5, 5.90)
- moved C2 0.30 mm to (26.3, 15.6)
Connections:
- net GND: now also X2.2, X2.3; no longer JP1.1, R3.1, X1.1, X1.4
- net N$4: now also X2.4; no longer X1.2
- net N$5: now also JP1.1; no longer R3.2, X1.3
- net N$6: now also X2.1; no longer JP1.2
Routing:
- net N$6: track 25.7 -> 23.1 mm
- net N$4: track 33.0 -> 31.5 mm
- net N$5: track 18.3 -> 18.9 mm, vias 2 -> 1
Other:
- board text added: "Vin GND GND Vout"
- board text removed: "GND Vout on/~off GND"
- board text removed: "Vin GND"
Changed lines of the file:
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@@
 <layer number="50" name="dxf" color="7" fill="1" visible="no" active="no"/>
 <layer number="51" name="tDocu" color="7" fill="1" visible="yes" active="yes"/>
-<layer number="52" name="bDocu" color="7" fill="1" visible="no" active="yes"/>
+<layer number="52" name="bDocu" color="7" fill="1" visible="yes" active="yes"/>
 <layer number="53" name="tGND_GNDA" color="7" fill="9" visible="no" active="no"/>
 <layer number="54" name="bGND_GNDA" color="1" fill="9" visible="no" active="no"/>
@@
 <wire x1="0" y1="23" x2="0" y2="0" width="0" layer="20"/>
 <hole x="3.1" y="20" drill="3.2"/>
-<text x="35.9" y="1.1" size="0.6096" layer="48" font="vector" rot="R90">GND
-Vout
-on/~off
-GND</text>
-<text x="35.8" y="16.2" size="0.6096" layer="48" font="vector" rot="R90">Vin
-GND</text>
+<text x="30.4" y="15" size="0.6096" layer="51" font="vector" rot="MR0">Vin
+GND
+GND
+Vout</text>
 </plain>
 <attributes>
@@
 <elements>
 <element name="IC1" library="Simplex-ICs" package="SO-08" value="LM2675M-ADJ" x="19.1" y="11.5"/>
-<element name="R1" library="rcl" package="R0805W" value="1.5K 1%" x="21.2" y="5.9" rot="R180"/>
-<element name="R2" library="rcl" package="R0805W" value="4.75k 1%" x="17" y="5.9" rot="R180"/>
+<element name="R1" library="rcl" package="R0805W" value="1.5K 1%" x="20.7" y="5.9" rot="R180"/>
+<element name="R2" library="rcl" package="R0805W" value="4.75k 1%" x="16.5" y="5.9" rot="R180"/>
 <element name="C1" library="rcl" package="C0805" value="10nF" x="15" y="11.5" rot="R90"/>
 <element name="D1" library="SparkFun-DiscreteSemi" package="SMA-DIODE" value="15MQ040" x="18.4" y="17.8" rot="R180">
 <attribute name="PROD_ID" value="DIO-08053" x="-1.92" y="33.04" size="1.778" layer="27" rot="R180" display="off"/>
 </element>
-<element name="C2" library="rcl" package="PANASONIC_F" value="47uF, 63V" x="26.6" y="15.6" rot="R90"/>
-<element name="C3" library="rcl" package="PANASONIC_D" value="100uF, 16V" x="26.7" y="5.8" rot="R270"/>
+<element name="C2" library="rcl" package="PANASONIC_F" value="47uF, 63V" x="26.3" y="15.6" rot="R90"/>
+<element name="C3" library="rcl" package="PANASONIC_D" value="100uF, 16V" x="26.1" y="5.8" rot="R270"/>
 <element name="L2" library="inductors" package="DR125" value="68uH 1.5A" x="7.2" y="10.2" rot="R270"/>
-<element name="JP1" library="SparkFun-Connectors" package="1X02" value="M02PTH" x="35.8" y="14" rot="R180"/>
-<element name="X1" library="Simplex-Connectors" package="0530480401" value="MOLEX_4HORIZONTAL" x="32.2" y="8"/>
-<element name="R3" library="rcl" package="R0805W" value="100k DNP" x="34.3" y="10.6" rot="R180"/>
+<element name="X2" library="con-phoenix-508" package="MKDSN1,5/4-5,08" value="MKDSN1,5/4-5,08" x="34.7" y="11.5" rot="R270">
+<attribute name="OC_NEWARK" value="70R0300" x="34.7" y="11.5" size="1.778" layer="27" rot="R270" display="off"/>
+<attribute name="MPN" value="SMKDSN1,5/4-5,08" x="34.7" y="11.5" size="1.778" layer="27" rot="R270" display="off"/>
+<attribute name="MF" value="" x="34.7" y="11.5" size="1.778" layer="27" rot="R270" display="off"/>
+<attribute name="OC_FARNELL" value="1792905" x="34.7" y="11.5" size="1.778" layer="27" rot="R270" display="off"/>
+</element>
+<element name="JP1" library="SparkFun-Connectors" package="1X01" value="M01PTH" x="29.1" y="1.5"/>
 </elements>
 <signals>
@@
 <vertex x="0" y="0"/>
 </polygon>
-<contactref element="JP1" pad="1"/>
-<contactref element="X1" pad="1"/>
-<contactref element="X1" pad="4"/>
-<contactref element="R3" pad="1"/>
 <via x="1" y="22" extent="1-16" drill="0.4"/>
 <via x="1" y="1" extent="1-16" drill="0.4"/>
@@
 <via x="13.2" y="22" extent="1-16" drill="0.4"/>
 <via x="13" y="1" extent="1-16" drill="0.4"/>
+<contactref element="X2" pad="2"/>
+<contactref element="X2" pad="3"/>
+<via x="21" y="10.9" extent="1-16" drill="0.4"/>
+<via x="17.2" y="12.1" extent="1-16" drill="0.4"/>
+<via x="17.2" y="10.9" extent="1-16" drill="0.4"/>
+<via x="21" y="12.1" extent="1-16" drill="0.4"/>
+<via x="23.7" y="12" extent="1-16" drill="0.4"/>
+<via x="23.7" y="8.2" extent="1-16" drill="0.4"/>
 </signal>
 <signal name="N$1">
@@
 <contactref element="IC1" pad="4"/>
 <contactref element="R2" pad="1"/>
-<wire x1="21.005" y1="8.9" x2="21.005" y2="7.305" width="0.4064" layer="1"/>
-<wire x1="21.005" y1="7.305" x2="20.3" y2="6.6" width="0.4064" layer="1"/>
-<wire x1="20.3" y1="6.6" x2="20.3" y2="6.0525" width="0.4064" layer="1"/>
-<wire x1="20.3" y1="6.0525" x2="20.1475" y2="5.9" width="0.4064" layer="1"/>
-<wire x1="18.0525" y1="5.9" x2="20.1475" y2="5.9" width="0.4064" layer="1"/>
+<wire x1="17.5525" y1="5.9" x2="19.6475" y2="5.9" width="0.4064" layer="1"/>
+<wire x1="19.6475" y1="5.9" x2="21.005" y2="7.2575" width="0.4064" layer="1"/>
+<wire x1="21.005" y1="7.2575" x2="21.005" y2="8.9" width="0.4064" layer="1"/>
 </signal>
 <signal name="N$2">
@@
 <contactref element="C3" pad="+"/>
 <contactref element="L2" pad="2"/>
-<contactref element="X1" pad="2"/>
-<wire x1="33.45" y1="8" x2="33.45" y2="5.25" width="1.016" layer="1"/>
-<wire x1="33.45" y1="5.25" x2="31.7" y2="3.5" width="1.016" layer="1"/>
-<wire x1="31.7" y1="3.5" x2="26.8" y2="3.5" width="1.016" layer="1"/>
-<wire x1="26.8" y1="3.5" x2="26.7" y2="3.4" width="1.016" layer="1"/>
+<wire x1="34.3239" y1="3.5" x2="26.8" y2="3.5" width="1.016" layer="1"/>
+<wire x1="26.8" y1="3.5" x2="26.1" y2="3.4" width="1.016" layer="1"/>
 <wire x1="7.2" y1="5.225" x2="9.025" y2="3.5" width="1.016" layer="1"/>
-<wire x1="9.025" y1="3.5" x2="16.1" y2="3.5" width="1.016" layer="1"/>
-<wire x1="16.1" y1="3.5" x2="26.8" y2="3.5" width="1.016" layer="1"/>
-<wire x1="15.9475" y1="5.9" x2="15.9475" y2="3.6525" width="0.4064" layer="1"/>
-<wire x1="15.9475" y1="3.6525" x2="16.1" y2="3.5" width="0.4064" layer="1"/>
+<wire x1="9.025" y1="3.5" x2="15.6" y2="3.5" width="1.016" layer="1"/>
+<wire x1="15.6" y1="3.5" x2="26.8" y2="3.5" width="1.016" layer="1"/>
+<wire x1="15.4475" y1="5.9" x2="15.4475" y2="3.6525" width="0.4064" layer="1"/>
+<wire x1="15.4475" y1="3.6525" x2="15.6" y2="3.5" width="0.4064" layer="1"/>
+<contactref element="X2" pad="4"/>
+<wire x1="34.3239" y1="3.5" x2="34.725" y2="3.9011" width="1.016" layer="1"/>
 </signal>
 <signal name="N$6">
@@
 <contactref element="C2" pad="+"/>
 <wire x1="18.465" y1="19.465" x2="18.465" y2="14.1" width="1.016" layer="1"/>
-<contactref element="JP1" pad="2"/>
-<wire x1="33.26" y1="14" x2="33.26" y2="17.34" width="1.016" layer="1"/>
-<wire x1="33.26" y1="17.34" x2="30.6" y2="20" width="1.016" layer="1"/>
 <wire x1="18.465" y1="19.465" x2="19" y2="20" width="1.016" layer="1"/>
 <wire x1="19" y1="20" x2="26.6" y2="20" width="1.016" layer="1"/>
-<wire x1="26.6" y1="20" x2="26.6" y2="19.15" width="1.016" layer="1"/>
-<wire x1="30.6" y1="20" x2="26.6" y2="20" width="1.016" layer="1"/>
+<wire x1="26.6" y1="20" x2="26.3" y2="19.15" width="1.016" layer="1"/>
+<wire x1="33.8661" y1="20" x2="26.6" y2="20" width="1.016" layer="1"/>
+<contactref element="X2" pad="1"/>
+<wire x1="33.8661" y1="20" x2="34.725" y2="19.1411" width="1.016" layer="1"/>
 </signal>
 <signal name="N$5">
 <contactref element="IC1" pad="5"/>
-<contactref element="X1" pad="3"/>
-<contactref element="R3" pad="2"/>
-<wire x1="33.2475" y1="10.6" x2="33.6" y2="10.6475" width="0.4064" layer="1"/>
-<via x="34" y="9.7" extent="1-16" drill="0.4"/>
-<wire x1="34" y1="9.7" x2="32.3" y2="11.3" width="0.4064" layer="16"/>
 <via x="22.6" y="13.1" extent="1-16" drill="0.4"/>
 <wire x1="21.005" y1="14.1" x2="22.005" y2="13.1" width="0.4064" layer="1"/>
 <wire x1="22.005" y1="13.1" x2="22.6" y2="13.1" width="0.4064" layer="1"/>
-<wire x1="32.3" y1="11.3" x2="24.4" y2="11.3" width="0.4064" layer="16"/>
-<wire x1="24.4" y1="11.3" x2="22.6" y2="13.1" width="0.4064" layer="16"/>
-<wire x1="34.7" y1="8" x2="34.7" y2="9" width="0.4064" layer="1"/>
-<wire x1="34.7" y1="9" x2="34" y2="9.7" width="0.4064" layer="1"/>
-<wire x1="34" y1="9.7" x2="33.2475" y2="10.4525" width="0.4064" layer="1"/>
-<wire x1="33.2475" y1="10.4525" x2="33.2475" y2="10.6" width="0.4064" layer="1"/>
+<contactref element="JP1" pad="1"/>
+<wire x1="22.6" y1="13.1" x2="22.6" y2="3.6" width="0.4064" layer="16"/>
+<wire x1="22.6" y1="3.6" x2="24.7" y2="1.5" width="0.4064" layer="16"/>
+<wire x1="24.7" y1="1.5" x2="29.1" y2="1.5" width="0.4064" layer="16"/>
 </signal>
 </signals>
